File: MainBoard.kicad_pcb (KiCad board)
At the start: 2 copper layers, 100 x 100 mm, 114 parts, among them J1 Conn_01x06, J10 Conn_01x02, J2 Conn_01x06, J3 Conn_01x02, J4 Conn_01x02, J5 Conn_01x02, J6 Conn_01x02, J7 Conn_01x03, J8 Conn_01x03, J9 Conn_01x05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

Commit message: Change routings&Add ESD for UART and CAN&Add 5V protection and pull-resistance for GPIO
Parts:
- added D5: BV03C, Diode_SMD:D_SOD-323, F.Cu at (217.9, 141.9)
- added D6: BV03C, Diode_SMD:D_SOD-323, F.Cu at (158.2, 126.6)
- added D7: 5V1, Diode_SMD:D_SOD-123, F.Cu at (235.4, 119.5)
- added R11: 1K, Resistor_SMD:R_0603_1608Metric, F.Cu at (241.9, 115.6)
- added R12: 1K, Resistor_SMD:R_0603_1608Metric, F.Cu at (241.9, 114.1)
- added R6: 1K, Resistor_SMD:R_0603_1608Metric, F.Cu at (241.9, 118.7)
- added R7: 1K, Resistor_SMD:R_0603_1608Metric, F.Cu at (241.9, 117.1)
- added U18: ~, Package_TO_SOT_SMD:SOT-23-3, F.Cu at (240.2, 80.0)
- added U19: ~, Package_TO_SOT_SMD:SOT-23-3, F.Cu at (240.2, 88.9)
- added U20: ~, Package_TO_SOT_SMD:SOT-23-3, F.Cu at (240.2, 106.7)
- added U21: ~, Package_TO_SOT_SMD:SOT-23-3, F.Cu at (240.2, 97.8)
- added U22: ~, Package_TO_SOT_SMD:SOT-23-5, F.Cu at (239.8, 140.2)
- J1, J2: value Conn_01x06 -> Conn_01x04; footprint Connector_FFC-FPC:Hirose_FH12-6S-0.5SH_1x06-1MP_P0.50mm_Horizontal -> Connector_Molex:Molex_CLIK-Mate_502386-0470_1x04-1MP_P1.25mm_Horizontal
- moved J1 60.0 mm to (224.2, 143.9)
- moved J2 59.7 mm to (164.0, 144.0)
- moved R16 18.4 mm to (232.8, 118.7)
- moved R17 15.5 mm to (231.3, 118.7)
- moved R18 7.23 mm to (224.7, 122.8), turned to 0 degrees
- moved C51 7.16 mm to (185.5, 133.7), turned to 180 degrees
- moved C43 6.44 mm to (170.0, 133.2), turned to -135 degrees
- moved R19 4.16 mm to (222.4, 123.5)
- moved R20 4.16 mm to (220.9, 123.5)
- moved R14 3.61 mm to (238.3, 145.2), turned to 90 degrees
- moved C16 3.60 mm to (219.4, 132.5)
- moved C15 3.43 mm to (219.4, 134.0)
- moved C48 2.98 mm to (184.5, 141.6), turned to 180 degrees
- moved C21 2.69 mm to (197.0, 120.2), turned to 0 degrees
- moved C8 2.64 mm to (181.1, 120.1), turned to 0 degrees
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Connections:
- J1 pad 1: unconnected-(J1-Pad1) -> /VBUS2
- J1 pad 2: unconnected-(J1-Pad2) -> /USB2-
- J1 pad 3: /VBUS1 -> /USB2+
- J1 pad 4: /USB1- -> GND
- J2 pad 1: unconnected-(J2-Pad1) -> /VBUS1
- J2 pad 2: unconnected-(J2-Pad2) -> /USB1-
- J2 pad 3: /VBUS2 -> /USB1+
- J2 pad 4: /USB2- -> GND
Routing:
- net /USB2CAN/3V3: track 347.8 -> 323.7 mm, vias 10 -> 0
- net /USB2CAN/STM2_CAN/USB_D+: track 49.9 -> 30.9 mm
- net /USB2CAN/STM2_CAN/USB_D-: track 51.0 -> 32.3 mm
- net /USB2GPIO/GPIO/SCL: track 37.1 -> 19.0 mm, vias 0 -> 2
- net /USB2GPIO/GPIO/SDA: track 36.3 -> 21.3 mm
- net /VBUS2: track 123.1 -> 108.5 mm, vias 5 -> 7
- net /VBUS1: track 121.0 -> 109.2 mm, vias 5 -> 4
- net Net-(U6-VDD18): track 13.8 -> 5.45 mm, vias 2 -> 0
- net /USB2GPIO/GPIO/*D-: track 10.9 -> 6.45 mm
- net Net-(U6-VDD33): track 10.8 -> 6.34 mm, vias 2 -> 0
- net /USB2GPIO/GPIO/*D+: track 10.3 -> 5.87 mm
- net /USB2GPIO/GPIO/D+: track 4.22 -> 8.14 mm
- net Net-(U12-VDD18): track 12.3 -> 9.34 mm, vias 2 -> 0
- net /USB1-: track 5.44 -> 7.83 mm
- net /USB1+: track 5.50 -> 7.90 mm
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Other:
- board text added: "0"
- board text added: "10K"
- board text added: "10u"
- board text added: "120"
- board text added: "18p"
- board text added: "1K"
- board text added: "2.2K"
- board text added: "4.7K"
- board text added: "47K"
- board text added: "68"
